Commit message: Initial commit of navigation for task 5, 9, 13.

File: walker_WAIC_18.04_v1.2_20200616/ubt_sim_ws/src/thewalkingdead/config/walker.urdf (robot description, URDF)
Before this commit: robot walker_description, 56 links, 55 joints
Links:
- added link boteye_imu_link
- added link boteye_link
- added link head_depth_link
- added link top_depth_link
Joints:
- added joint base_boteye_imu: type fixed, parent base_link, child boteye_imu_link, origin xyz=0 0 0 rpy=0 0 0
- added joint base_boteye_link: type fixed, parent base_link, child boteye_link, origin xyz=0 0 0 rpy=0 0 0
- added joint base_head_depth: type fixed, parent base_link, child head_depth_link, origin xyz=0 0.3229 0 rpy=0 -0.349 0
- added joint base_top_depth: type fixed, parent base_link, child top_depth_link, origin xyz=0 0 0 rpy=0 0 0

Commit message: Merging IMU with VO

File: walker_WAIC_18.04_v1.2_20200616/ubt_sim_ws/src/thewalkingdead/config/walker.urdf (robot description, URDF)
Before this commit: robot walker_description, 60 links, 59 joints
Links:
- added link head_imu_link
- added link orientus_imu_link
Joints:
- added joint base_head_imu: type fixed, parent base_link, child head_imu_link, origin xyz=0 0.3229 0 rpy=0 0 1.5708
- added joint base_orientus_imu: type fixed, parent base_link, child orientus_imu_link, origin xyz=0 -0.2321 0 rpy=0 0 1.5708
- joint base_boteye_imu: origin xyz=0 0 0 rpy=0 0 0 -> xyz=0 0 0 rpy=0 0 1.5708
